Commit message: fix(nav2): add laser range filter to eliminate chassis self-reflections
RPLIDAR C1 sees ~145 scan points from robot chassis at 0.02-0.09m range,
which slam_toolbox bakes into the map as permanent obstacles at the robot
position, causing Nav2 planner "Start occupied" errors.

- Add laser_filter.yaml: LaserScanRangeFilter drops returns < 0.15m
- Modify robot.launch.py: sllidar publishes /scan_raw, laser_filter_node
  filters and republishes as /scan
- Fix URDF laser joint: add pi yaw for 180-deg mounted RPLIDAR
- Add rviz2 Tools section: 2D Goal Pose, SetInitialPose, etc.
- Set obstacle_min_range: 0.20 on both costmap obstacle layers

Co-Authored-By: Claude Opus 4.6 <noreply@anthropic.com>

File: roscar_ws/src/roscar_description/urdf/roscar.urdf.xacro (robot description, xacro)
@@ -128,5 +128,5 @@
     <parent link="base_link"/>
     <child link="laser"/>
-    <origin xyz="${lidar_x} 0 ${lidar_z}" rpy="0 0 0"/>
+    <origin xyz="${lidar_x} 0 ${lidar_z}" rpy="0 0 ${pi}"/>
   </joint>
 </robot>

Commit message: feat: update for top-mounted lidar — remove laser filter
Lidar moved from middle platform to top platform with clear 360-degree
view. Updated URDF lidar_z (0.12→0.09), removed laser_filter_node from
robot.launch.py (no more chassis self-reflections), and reset costmap
obstacle_min_range to 0.0.

Co-Authored-By: Claude Opus 4.6 <noreply@anthropic.com>

File: roscar_ws/src/roscar_description/urdf/roscar.urdf.xacro (robot description, xacro)
@@ -17,5 +17,5 @@
   <!-- Lidar position (relative to base_link) -->
   <xacro:property name="lidar_x" value="0.0"/>
-  <xacro:property name="lidar_z" value="0.12"/>  <!-- top of chassis -->
+  <xacro:property name="lidar_z" value="0.09"/>  <!-- top platform, scan plane ~18cm from floor -->
   <!-- ==================== Materials ==================== -->
   <material name="dark_grey">

Commit message: description: rename webcam link, add D435i via realsense2_description xacro
- rename camera_link/camera_optical_frame -> webcam_link/webcam_optical_frame
  to free the 'camera_link' name for realsense2_description's D435i macro
- include sensor_d435i macro mounted at front of chassis, tilted 10deg down
  (d435i_x/y/z/pitch placeholders; measure and update after physical mount)
- update camera.launch.py to set frame_id='webcam_optical_frame'
- update aruco_detector_node.py frame references
- update landmark_localizer_node.py TF lookups and docstring

Co-Authored-By: Claude Opus 4.7 (1M context) <noreply@anthropic.com>

File: roscar_ws/src/roscar_description/urdf/roscar.urdf.xacro (robot description, xacro)
@@ -1,4 +1,6 @@
 <?xml version="1.0"?>
 <robot xmlns:xacro="http://www.ros.org/wiki/xacro" name="roscar">
+  <!-- Include D435i macro from realsense2_description -->
+  <xacro:include filename="$(find realsense2_description)/urdf/_d435i.urdf.xacro"/>
   <!-- ==================== Robot Dimensions ==================== -->
   <!-- MEASURED 2026-03-16 with calipers and tape measure            -->
@@ -18,4 +20,10 @@
   <xacro:property name="lidar_x" value="0.0"/>
   <xacro:property name="lidar_z" value="0.09"/>  <!-- scan plane ~18cm from floor -->
+  <!-- D435i depth camera position (relative to base_link) — front-facing, tilted slightly down -->
+  <!-- TODO: measure after physical mount — placeholder values below -->
+  <xacro:property name="d435i_x" value="0.09"/>    <!-- m, forward of center -->
+  <xacro:property name="d435i_y" value="0.0"/>     <!-- m, centered -->
+  <xacro:property name="d435i_z" value="0.07"/>    <!-- m, above base_link -->
+  <xacro:property name="d435i_pitch" value="0.175"/>  <!-- rad, ~10deg down tilt -->
   <!-- ==================== Materials ==================== -->
   <material name="dark_grey">
@@ -95,6 +103,9 @@
     <origin xyz="0 0 0" rpy="0 0 0"/>
   </joint>
-  <!-- ==================== Camera Link ==================== -->
-  <link name="camera_link">
+  <!-- ==================== Logitech Webcam Link ==================== -->
+  <!-- NOTE: renamed from camera_link to webcam_link to free the "camera_link"
+       name for realsense2_description's D435i macro (below). Any consumer that
+       used camera_optical_frame should use webcam_optical_frame now. -->
+  <link name="webcam_link">
     <visual>
       <geometry>
@@ -104,16 +115,24 @@
     </visual>
   </link>
-  <joint name="camera_joint" type="fixed">
+  <joint name="webcam_joint" type="fixed">
     <parent link="base_link"/>
-    <child link="camera_link"/>
+    <child link="webcam_link"/>
     <origin xyz="${camera_x} 0 ${camera_z}" rpy="0 0 0"/>
   </joint>
   <!-- Optical frame: z forward, x right, y down (REP 103) -->
-  <link name="camera_optical_frame"/>
-  <joint name="camera_optical_joint" type="fixed">
-    <parent link="camera_link"/>
-    <child link="camera_optical_frame"/>
+  <link name="webcam_optical_frame"/>
+  <joint name="webcam_optical_joint" type="fixed">
+    <parent link="webcam_link"/>
+    <child link="webcam_optical_frame"/>
     <origin xyz="0 0 0" rpy="${-pi/2} 0 ${-pi/2}"/>
   </joint>
+  <!-- ==================== D435i Depth Camera ==================== -->
+  <!-- realsense2_description's sensor_d435i macro creates:
+         camera_link (body), camera_depth_frame, camera_color_frame,
+         camera_accel_frame, camera_gyro_frame, and their _optical variants.
+       Parented to base_link at the mount pose defined above. -->
+  <xacro:sensor_d435i parent="base_link" name="camera" use_nominal_extrinsics="true">
+    <origin xyz="${d435i_x} ${d435i_y} ${d435i_z}" rpy="0 ${d435i_pitch} 0"/>
+  </xacro:sensor_d435i>
   <!-- ==================== Lidar Link (RPLIDAR C1) ==================== -->
   <link name="laser">

Commit message: d435i: replace Logitech webcam outright, consolidate to single camera
The D435i now serves both jobs: depth pointcloud (Nav2 voxel_layer) AND
color stream (dashboard, ArUco, YOLO). One sensor, one USB port, one set
of TF frames. Color stream is factory-calibrated and global-shutter
(better for marker detection than the Logitech's rolling shutter).

Changes:
- robot.launch.py: use_camera default true -> false (legacy webcam opt-in
  only); use_depth default false -> true (D435i is primary camera now)
- depth_camera.launch.py: remap /camera/camera/color/image_raw -> /image_raw
  and /camera/camera/color/camera_info -> /camera_info so dashboard MJPEG
  stream, ArUco detector, and YOLO need zero config changes
- realsense_params.yaml: color profile 640x480@15 -> 640x480@30 (USB 3.0
  has headroom, dashboard+CV prefer 30)
- aruco_detector_node.py: marker TF frame_id camera_optical_frame (was
  webcam_optical_frame briefly) -> camera_color_optical_frame (D435i's
  factory-provided optical frame)
- landmark_localizer_node.py: TF lookup map -> camera_color_optical_frame
- roscar.urdf.xacro: removed webcam_link / webcam_optical_frame block
  (8 lines + 2 properties). camera_link now unambiguously refers to the
  D435i's body frame

Verified on Pi5 after fresh boot:
- /image_raw at 28.6 Hz, publisher = realsense driver ✓
- /camera/camera/depth/color/points at 15.4 Hz ✓
- base_link -> camera_color_optical_frame translation (0.103, 0.032, 0.080),
  camera +z points (0.985, 0, -0.174) in base_link = 10deg down tilt ✓
- No v4l2_camera_node spawned (use_camera=false working) ✓
- URDF has 0 webcam references ✓

Co-Authored-By: Claude Opus 4.7 (1M context) <noreply@anthropic.com>

File: roscar_ws/src/roscar_description/urdf/roscar.urdf.xacro (robot description, xacro)
@@ -14,7 +14,4 @@
   <xacro:property name="wheel_x_offset" value="0.0483"/>  <!-- m, half of 96.55mm wheelbase -->
   <xacro:property name="wheel_y_offset" value="0.1025"/>  <!-- m, half of 205mm track width -->
-  <!-- Camera position (relative to base_link) — TODO: measure precisely -->
-  <xacro:property name="camera_x" value="0.12"/>
-  <xacro:property name="camera_z" value="0.10"/>
   <!-- Lidar position (relative to base_link) — TODO: measure precisely -->
   <xacro:property name="lidar_x" value="0.0"/>
@@ -103,28 +100,4 @@
     <origin xyz="0 0 0" rpy="0 0 0"/>
   </joint>
-  <!-- ==================== Logitech Webcam Link ==================== -->
-  <!-- NOTE: renamed from camera_link to webcam_link to free the "camera_link"
-       name for realsense2_description's D435i macro (below). Any consumer that
-       used camera_optical_frame should use webcam_optical_frame now. -->
-  <link name="webcam_link">
-    <visual>
-      <geometry>
-        <box size="0.03 0.08 0.03"/>
-      </geometry>
-      <material name="blue"/>
-    </visual>
-  </link>
-  <joint name="webcam_joint" type="fixed">
-    <parent link="base_link"/>
-    <child link="webcam_link"/>
-    <origin xyz="${camera_x} 0 ${camera_z}" rpy="0 0 0"/>
-  </joint>
-  <!-- Optical frame: z forward, x right, y down (REP 103) -->
-  <link name="webcam_optical_frame"/>
-  <joint name="webcam_optical_joint" type="fixed">
-    <parent link="webcam_link"/>
-    <child link="webcam_optical_frame"/>
-    <origin xyz="0 0 0" rpy="${-pi/2} 0 ${-pi/2}"/>
-  </joint>
   <!-- ==================== D435i Depth Camera ==================== -->
   <!-- realsense2_description's sensor_d435i macro creates:

Commit message: urdf+cv: extrusion-chassis mast model + WSL2 CV systemd unit
URDF reflects the rebuilt aluminum-extrusion chassis: 3030 mast at +X
holding the D435i and RPLIDAR C1 on top. Wheelbase/track/heights are
estimates marked TODO until measured. Material renamed to
roscar_aluminum to avoid clash with realsense2_description.

scripts/roscar-cv.sh + roscar-cv.service mirror the Pi's roscar-web
pattern so the CV stack (ArUco + YOLO + cv_video_server) survives
WSL2 reboots.

Co-Authored-By: Claude Opus 4.7 (1M context) <noreply@anthropic.com>

File: roscar_ws/src/roscar_description/urdf/roscar.urdf.xacro (robot description, xacro)
@@ -1,24 +1,45 @@
 <?xml version="1.0"?>
 <robot xmlns:xacro="http://www.ros.org/wiki/xacro" name="roscar">
-  <!-- ==================== Robot Dimensions ==================== -->
-  <!-- MEASURED 2026-03-16 with calipers and tape measure            -->
-  <xacro:property name="chassis_length" value="0.200"/>   <!-- m, front-to-back (body, not incl wheel protrusion) -->
-  <xacro:property name="chassis_width" value="0.170"/>    <!-- m, left-to-right (body between wheels) -->
-  <xacro:property name="chassis_height" value="0.060"/>   <!-- m, plate/board stack thickness -->
-  <xacro:property name="chassis_z_offset" value="0.0205"/> <!-- m, ground to bottom of chassis (measured) -->
-  <xacro:property name="wheel_radius" value="0.0397"/>    <!-- m, 79.3mm dia across mecanum rollers -->
-  <xacro:property name="wheel_width" value="0.0373"/>     <!-- m, hub face to face incl rollers -->
-  <!-- Half-distances from center to wheel axes -->
-  <xacro:property name="wheel_x_offset" value="0.0483"/>  <!-- m, half of 96.55mm wheelbase -->
-  <xacro:property name="wheel_y_offset" value="0.1025"/>  <!-- m, half of 205mm track width -->
-  <!-- Camera position (relative to base_link) — TODO: measure precisely -->
-  <xacro:property name="camera_x" value="0.12"/>
-  <xacro:property name="camera_z" value="0.10"/>
-  <!-- Lidar position (relative to base_link) — TODO: measure precisely -->
-  <xacro:property name="lidar_x" value="0.0"/>
-  <xacro:property name="lidar_z" value="0.09"/>  <!-- scan plane ~18cm from floor -->
+  <!-- Include D435i macro from realsense2_description -->
+  <xacro:include filename="$(find realsense2_description)/urdf/_d435i.urdf.xacro"/>
+  <!-- ==================== Coordinate Convention ==================== -->
+  <!-- base_link: +X = camera mast direction (operator forward), +Y = left,    -->
+  <!-- +Z = up (REP 103). Driver runs no vx/vy negation in this state — motor  -->
+  <!-- wiring matches firmware labels and base_link aligns with the firmware   -->
+  <!-- chassis frame.                                                          -->
+  <!-- ==================== Robot Dimensions (Chassis v2 — extrusion) ============ -->
+  <!-- ESTIMATES from photos 2026-04-27. TODO: remeasure with calipers/tape:    -->
+  <!--   wheelbase, track, mast_x, mast_height, d435i_z, lidar_z.               -->
+  <xacro:property name="chassis_length" value="0.220"/>   <!-- ESTIMATE -->
+  <xacro:property name="chassis_width"  value="0.220"/>   <!-- ESTIMATE -->
+  <xacro:property name="chassis_height" value="0.080"/>   <!-- ESTIMATE: extrusion stack -->
+  <xacro:property name="chassis_z_offset" value="0.0205"/> <!-- ground to bottom of frame -->
+  <xacro:property name="wheel_radius" value="0.0397"/>    <!-- 79.3mm dia mecanum -->
+  <xacro:property name="wheel_width"  value="0.0373"/>
+  <!-- Half-distances from chassis center to wheel hubs.                       -->
+  <!-- ESTIMATE — please measure: hub-to-hub fore/aft = 2*wheel_x_offset,      -->
+  <!-- hub-to-hub left/right = 2*wheel_y_offset.                                -->
+  <xacro:property name="wheel_x_offset" value="0.085"/>   <!-- ESTIMATE: half wheelbase ~170mm -->
+  <xacro:property name="wheel_y_offset" value="0.110"/>   <!-- ESTIMATE: half track ~220mm -->
+  <!-- Mast (3030 extrusion column at front of chassis, holds lidar + camera) -->
+  <xacro:property name="mast_x"        value="0.090"/>    <!-- ESTIMATE: forward of base_link center -->
+  <xacro:property name="mast_height"   value="0.220"/>    <!-- ESTIMATE: column length above chassis top -->
+  <xacro:property name="mast_section"  value="0.030"/>    <!-- 30mm extrusion -->
+  <!-- D435i camera mounted on the front face of the mast, looking +X.        -->
+  <!-- ESTIMATE — please measure ground to camera optical-center height.       -->
+  <xacro:property name="d435i_x"     value="${mast_x + mast_section/2}"/>
+  <xacro:property name="d435i_y"     value="0.0"/>
+  <xacro:property name="d435i_z"     value="0.150"/>      <!-- ESTIMATE: above base_link -->
+  <xacro:property name="d435i_pitch" value="0.0"/>        <!-- horizontal -->
+  <!-- Lidar sits on top of the mast.                                          -->
+  <!-- ESTIMATE — please measure ground to scan-plane height.                  -->
+  <xacro:property name="lidar_x" value="${mast_x}"/>
+  <xacro:property name="lidar_z" value="${mast_height + 0.015}"/>  <!-- mast top + ~15mm to scan plane -->
   <!-- ==================== Materials ==================== -->
   <material name="dark_grey">
     <color rgba="0.3 0.3 0.3 1.0"/>
+  </material>
+  <material name="roscar_aluminum">
+    <color rgba="0.75 0.75 0.78 1.0"/>
   </material>
   <material name="black">
@@ -29,5 +50,4 @@
   </material>
   <!-- ==================== Base Footprint ==================== -->
-  <!-- Virtual frame on the ground plane, directly below base_link -->
   <link name="base_footprint"/>
   <joint name="base_footprint_joint" type="fixed">
@@ -50,8 +70,23 @@
     </collision>
     <inertial>
-      <mass value="2.2"/>  <!-- measured total 2200g, minus ~400g for 4 wheels -->
-      <inertia ixx="0.01" ixy="0" ixz="0" iyy="0.01" iyz="0" izz="0.01"/>
+      <mass value="3.5"/>  <!-- ESTIMATE: extrusion frame ~3-4kg total -->
+      <inertia ixx="0.02" ixy="0" ixz="0" iyy="0.02" iyz="0" izz="0.02"/>
     </inertial>
   </link>
+  <!-- ==================== Camera Mast (3030 extrusion column) ============== -->
+  <link name="mast_link">
+    <visual>
+      <origin xyz="0 0 ${mast_height/2}" rpy="0 0 0"/>
+      <geometry>
+        <box size="${mast_section} ${mast_section} ${mast_height}"/>
+      </geometry>
+      <material name="roscar_aluminum"/>
+    </visual>
+  </link>
+  <joint name="mast_joint" type="fixed">
+    <parent link="base_link"/>
+    <child link="mast_link"/>
+    <origin xyz="${mast_x} 0 ${chassis_height/2}" rpy="0 0 0"/>
+  </joint>
   <!-- ==================== Wheel Macro ==================== -->
   <xacro:macro name="mecanum_wheel" params="name x_pos y_pos">
@@ -95,30 +130,18 @@
     <origin xyz="0 0 0" rpy="0 0 0"/>
   </joint>
-  <!-- ==================== Camera Link ==================== -->
-  <link name="camera_link">
-    <visual>
-      <geometry>
-        <box size="0.03 0.08 0.03"/>
-      </geometry>
-      <material name="blue"/>
-    </visual>
-  </link>
-  <joint name="camera_joint" type="fixed">
-    <parent link="base_link"/>
-    <child link="camera_link"/>
-    <origin xyz="${camera_x} 0 ${camera_z}" rpy="0 0 0"/>
-  </joint>
-  <!-- Optical frame: z forward, x right, y down (REP 103) -->
-  <link name="camera_optical_frame"/>
-  <joint name="camera_optical_joint" type="fixed">
-    <parent link="camera_link"/>
-    <child link="camera_optical_frame"/>
-    <origin xyz="0 0 0" rpy="${-pi/2} 0 ${-pi/2}"/>
-  </joint>
-  <!-- ==================== Lidar Link (RPLIDAR C1) ==================== -->
+  <!-- ==================== D435i Depth Camera (mounted on mast) ============== -->
+  <!-- realsense2_description's sensor_d435i macro creates camera_link plus    -->
+  <!-- depth/color/IR child frames and their _optical variants. Parented to    -->
+  <!-- base_link at the mount pose; the macro handles internal extrinsics.     -->
+  <xacro:sensor_d435i parent="base_link" name="camera" use_nominal_extrinsics="true">
+    <origin xyz="${d435i_x} ${d435i_y} ${d435i_z}" rpy="0 ${d435i_pitch} 0"/>
+  </xacro:sensor_d435i>
+  <!-- ==================== Lidar Link (RPLIDAR C1, on top of mast) ========== -->
+  <!-- yaw=0: assumes the lidar's 0 deg marker points +X (toward camera direction). -->
+  <!-- If obstacles in front of the robot show up at -X in /scan, change to pi.     -->
   <link name="laser">
     <visual>
       <geometry>
-        <cylinder radius="0.035" length="0.025"/>
+        <cylinder radius="0.035" length="0.040"/>
       </geometry>
       <material name="blue"/>
@@ -128,5 +151,5 @@
     <parent link="base_link"/>
     <child link="laser"/>
-    <origin xyz="${lidar_x} 0 ${lidar_z}" rpy="0 0 ${pi}"/>
+    <origin xyz="${lidar_x} 0 ${lidar_z}" rpy="0 0 0"/>
   </joint>
 </robot>

Commit message: chassis v2 tuning: measured dims + scan-driven SLAM + AMCL auto-seed
Wheelbase + track measured (213mm × 325mm vs old 96mm × 205mm — the
firmware's mecanum FK overstates wz by ~1.8x with stale constants).
URDF wheel offsets, chassis width, and mast offset (15mm left of
center) updated to match. Lidar yaw flipped to π — physical 0° marker
points -X away from camera, verified empirically when scan-matcher
inferred backward motion under forward driving.

To kill the wavy-walls drift on carpet (where mecanum wheel slip is
significant), drop wheel vx/vy and wz from EKF entirely and let
slam_toolbox carry the full pose. Pre-requisite: switch slam_toolbox
to time-only triggering (minimum_travel_distance/heading = 0) so it
keeps firing even when EKF reports zero motion.

AMCL set_initial_pose: true so nav mode auto-seeds at origin on
activation instead of needing a manual /initialpose publish.

Driver twist covariance vx/vy bumped 0.01→0.25 — moot now that EKF
drops the channel, kept as documentation that wheel velocity reports
are not trusted on this chassis.

Co-Authored-By: Claude Opus 4.7 (1M context) <noreply@anthropic.com>

File: roscar_ws/src/roscar_description/urdf/roscar.urdf.xacro (robot description, xacro)
@@ -12,5 +12,5 @@
   <!--   wheelbase, track, mast_x, mast_height, d435i_z, lidar_z.               -->
   <xacro:property name="chassis_length" value="0.220"/>   <!-- ESTIMATE -->
-  <xacro:property name="chassis_width"  value="0.220"/>   <!-- ESTIMATE -->
+  <xacro:property name="chassis_width"  value="0.250"/>   <!-- MEASURED 2026-04-28: 250mm extrusion frame width -->
   <xacro:property name="chassis_height" value="0.080"/>   <!-- ESTIMATE: extrusion stack -->
   <xacro:property name="chassis_z_offset" value="0.0205"/> <!-- ground to bottom of frame -->
@@ -18,10 +18,11 @@
   <xacro:property name="wheel_width"  value="0.0373"/>
   <!-- Half-distances from chassis center to wheel hubs.                       -->
-  <!-- ESTIMATE — please measure: hub-to-hub fore/aft = 2*wheel_x_offset,      -->
-  <!-- hub-to-hub left/right = 2*wheel_y_offset.                                -->
-  <xacro:property name="wheel_x_offset" value="0.085"/>   <!-- ESTIMATE: half wheelbase ~170mm -->
-  <xacro:property name="wheel_y_offset" value="0.110"/>   <!-- ESTIMATE: half track ~220mm -->
+  <!-- MEASURED 2026-04-28: wheelbase 213mm (76mm rear-of-frame→rear-wheel,    -->
+  <!-- 289mm rear-of-frame→front-wheel), track 325mm.                          -->
+  <xacro:property name="wheel_x_offset" value="0.1065"/>  <!-- half wheelbase 213mm -->
+  <xacro:property name="wheel_y_offset" value="0.1625"/>  <!-- half track 325mm -->
   <!-- Mast (3030 extrusion column at front of chassis, holds lidar + camera) -->
   <xacro:property name="mast_x"        value="0.090"/>    <!-- ESTIMATE: forward of base_link center -->
+  <xacro:property name="mast_y"        value="0.015"/>    <!-- MEASURED 2026-04-28: 110mm from left edge of 250mm frame → 15mm left of center -->
   <xacro:property name="mast_height"   value="0.220"/>    <!-- ESTIMATE: column length above chassis top -->
   <xacro:property name="mast_section"  value="0.030"/>    <!-- 30mm extrusion -->
@@ -29,5 +30,5 @@
   <!-- ESTIMATE — please measure ground to camera optical-center height.       -->
   <xacro:property name="d435i_x"     value="${mast_x + mast_section/2}"/>
-  <xacro:property name="d435i_y"     value="0.0"/>
+  <xacro:property name="d435i_y"     value="${mast_y}"/>
   <xacro:property name="d435i_z"     value="0.150"/>      <!-- ESTIMATE: above base_link -->
   <xacro:property name="d435i_pitch" value="0.0"/>        <!-- horizontal -->
@@ -35,4 +36,5 @@
   <!-- ESTIMATE — please measure ground to scan-plane height.                  -->
   <xacro:property name="lidar_x" value="${mast_x}"/>
+  <xacro:property name="lidar_y" value="${mast_y}"/>
   <xacro:property name="lidar_z" value="${mast_height + 0.015}"/>  <!-- mast top + ~15mm to scan plane -->
   <!-- ==================== Materials ==================== -->
@@ -87,5 +89,5 @@
     <parent link="base_link"/>
     <child link="mast_link"/>
-    <origin xyz="${mast_x} 0 ${chassis_height/2}" rpy="0 0 0"/>
+    <origin xyz="${mast_x} ${mast_y} ${chassis_height/2}" rpy="0 0 0"/>
   </joint>
   <!-- ==================== Wheel Macro ==================== -->
@@ -138,6 +140,7 @@
   </xacro:sensor_d435i>
   <!-- ==================== Lidar Link (RPLIDAR C1, on top of mast) ========== -->
-  <!-- yaw=0: assumes the lidar's 0 deg marker points +X (toward camera direction). -->
-  <!-- If obstacles in front of the robot show up at -X in /scan, change to pi.     -->
+  <!-- yaw=π: lidar's 0 deg marker physically points -X (away from camera).        -->
+  <!-- Verified empirically 2026-04-28 — with yaw=0 the scan-matcher inferred      -->
+  <!-- backward motion when the robot drove forward.                               -->
   <link name="laser">
     <visual>
@@ -151,5 +154,5 @@
     <parent link="base_link"/>
     <child link="laser"/>
-    <origin xyz="${lidar_x} 0 ${lidar_z}" rpy="0 0 0"/>
+    <origin xyz="${lidar_x} ${lidar_y} ${lidar_z}" rpy="0 0 ${pi}"/>
   </joint>
 </robot>
